File: pcb/wifisign.sch (KiCad schematic (older format))
At the start: 19 parts, among them K1 CONN_3, K2 CONN_3, P1 CONN_2, P2 CONN_4, P3 CONN_1, P4 CONN_1, Q1 MOS_N, Q2 MOS_N, SW1 SW_PUSH, SW2 SW_PUSH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

Commit message: Wider output lines and boot pin changed to jumper
Parts:
- removed P3: CONN_1, symbol CONN_1
- added JP1: JUMPER, symbol JUMPER
Connections:
- net GND: now also JP1.1
- net at R2.2, U1.14 (GPIO0): now also JP1.2
Changed lines of the file:
@@
-EESchema Schematic File Version 2  date So 10. október 2015, 12:41:05 CEST
+EESchema Schematic File Version 2  date Po 12. október 2015, 13:07:20 CEST
 LIBS:power
 LIBS:device
@@
 Sheet 1 1
 Title ""
-Date "10 oct 2015"
+Date "12 oct 2015"
 Rev ""
 Comp ""
@@
 $EndDescr
 Wire Wire Line
+	1950 2900 1950 3000
+Wire Wire Line
 	2100 3400 2950 3400
 Wire Wire Line
@@
 Wire Wire Line
 	5100 3250 4850 3250
-Wire Wire Line
-	2600 2900 4900 2900
 Wire Wire Line
 	3700 3400 3300 3400
@@
 Connection ~ 7850 3300
 Wire Wire Line
-	4900 2900 4900 3150
+	4900 3150 4900 2900
 Connection ~ 4900 3150
 Wire Wire Line
@@
 Wire Wire Line
 	2100 3500 3700 3500
+Wire Wire Line
+	4900 2900 2550 2900
 $Comp
 L GND #PWR01
+U 1 1 561B943B
+P 1950 3000
+F 0 "#PWR01" H 1950 3000 30  0001 C CNN
+F 1 "GND" H 1950 2930 30  0001 C CNN
+	1    1950 3000
+	1    0    0    -1
+$EndComp
+$Comp
+L JUMPER JP1
+U 1 1 561B942B
+P 2250 2900
+F 0 "JP1" H 2250 3050 60  0000 C CNN
+F 1 "JUMPER" H 2250 2820 40  0000 C CNN
+	1    2250 2900
+	1    0    0    -1
+$EndComp
+$Comp
+L GND #PWR02
 U 1 1 5614CC0B
 P 2850 4600
-F 0 "#PWR01" H 2850 4600 30  0001 C CNN
+F 0 "#PWR02" H 2850 4600 30  0001 C CNN
 F 1 "GND" H 2850 4530 30  0001 C CNN
 	1    2850 4600
@@
 $EndComp
 $Comp
-L CONN_1 P3
-U 1 1 5614C7A3
-P 2450 2900
-F 0 "P3" H 2530 2900 40  0000 L CNN
-F 1 "CONN_1" H 2450 2955 30  0001 C CNN
-	1    2450 2900
-	-1   0    0    1
-$EndComp
-$Comp
 L CONN_4 P2
 U 1 1 5614C4E8
@@
 $EndComp
 $Comp
-L GND #PWR02
+L GND #PWR03
 U 1 1 5612672C
 P 6600 2600
-F 0 "#PWR02" H 6600 2600 30  0001 C CNN
+F 0 "#PWR03" H 6600 2600 30  0001 C CNN
 F 1 "GND" H 6600 2530 30  0001 C CNN
 	1    6600 2600
@@
 $EndComp
 $Comp
-L GND #PWR03
+L GND #PWR04
 U 1 1 56126634
 P 5650 4200
-F 0 "#PWR03" H 5650 4200 30  0001 C CNN
+F 0 "#PWR04" H 5650 4200 30  0001 C CNN
 F 1 "GND" H 5650 4130 30  0001 C CNN
 	1    5650 4200
@@
 $EndComp
 $Comp
-L GND #PWR04
+L GND #PWR05
 U 1 1 56126568
 P 7850 4150
-F 0 "#PWR04" H 7850 4150 30  0001 C CNN
+F 0 "#PWR05" H 7850 4150 30  0001 C CNN
 F 1 "GND" H 7850 4080 30  0001 C CNN
 	1    7850 4150
@@
 $EndComp
 $Comp
-L GND #PWR05
+L GND #PWR06
 U 1 1 56126563
 P 7300 4150
-F 0 "#PWR05" H 7300 4150 30  0001 C CNN
+F 0 "#PWR06" H 7300 4150 30  0001 C CNN
 F 1 "GND" H 7300 4080 30  0001 C CNN
 	1    7300 4150
@@
 $EndComp
 $Comp
-L GND #PWR06
+L GND #PWR07
 U 1 1 56126554
 P 7200 3200
-F 0 "#PWR06" H 7200 3200 30  0001 C CNN
+F 0 "#PWR07" H 7200 3200 30  0001 C CNN
 F 1 "GND" H 7200 3130 30  0001 C CNN
 	1    7200 3200
@@
 $EndComp
 $Comp
-L GND #PWR07
+L GND #PWR08
 U 1 1 56126465
 P 5600 3500
-F 0 "#PWR07" H 5600 3500 30  0001 C CNN
+F 0 "#PWR08" H 5600 3500 30  0001 C CNN
 F 1 "GND" H 5600 3430 30  0001 C CNN
 	1    5600 3500
@@
 $EndComp
 $Comp
-L +3.3V #PWR08
+L +3.3V #PWR09
 U 1 1 561263CA
 P 5600 3000
-F 0 "#PWR08" H 5600 2960 30  0001 C CNN
+F 0 "#PWR09" H 5600 2960 30  0001 C CNN
 F 1 "+3.3V" H 5600 3110 30  0000 C CNN
 	1    5600 3000
@@
 $EndComp
 $Comp
-L GND #PWR09
+L GND #PWR010
 U 1 1 56126336
 P 2550 2300
-F 0 "#PWR09" H 2550 2300 30  0001 C CNN
+F 0 "#PWR010" H 2550 2300 30  0001 C CNN
 F 1 "GND" H 2550 2230 30  0001 C CNN
 	1    2550 2300
@@
 $EndComp
 $Comp
-L GND #PWR010
+L GND #PWR011
 U 1 1 561262F8
 P 3500 3300
-F 0 "#PWR010" H 3500 3300 30  0001 C CNN
+F 0 "#PWR011" H 3500 3300 30  0001 C CNN
 F 1 "GND" H 3500 3230 30  0001 C CNN
 	1    3500 3300
@@
 $EndComp
 $Comp
-L +3.3V #PWR011
+L +3.3V #PWR012
 U 1 1 561262F2
 P 3500 3100
-F 0 "#PWR011" H 3500 3060 30  0001 C CNN
+F 0 "#PWR012" H 3500 3060 30  0001 C CNN
 F 1 "+3.3V" H 3500 3210 30  0000 C CNN
 	1    3500 3100
@@
 $EndComp
 $Comp
-L +3.3V #PWR012
+L +3.3V #PWR013
 U 1 1 561262CC
 P 2550 1350
-F 0 "#PWR012" H 2550 1310 30  0001 C CNN
+F 0 "#PWR013" H 2550 1310 30  0001 C CNN
 F 1 "+3.3V" H 2550 1460 30  0000 C CNN
 	1    2550 1350
@@
 $EndComp
 $Comp
-L GND #PWR013
+L GND #PWR014
 U 1 1 561262BF
 P 1150 1900
-F 0 "#PWR013" H 1150 1900 30  0001 C CNN
+F 0 "#PWR014" H 1150 1900 30  0001 C CNN
 F 1 "GND" H 1150 1830 30  0001 C CNN
 	1    1150 1900

Commit message: Fixed board
Connections:
- net +3.3V: now also K1.2 (PM), K2.1 (P1)
- net GND: no longer K1.2 (PM), K2.1 (P1)
Changed lines of the file:
@@
-EESchema Schematic File Version 2  date Po 12. október 2015, 13:07:20 CEST
+EESchema Schematic File Version 2  date Št 15. október 2015, 10:42:44 CEST
 LIBS:power
 LIBS:device
@@
 Sheet 1 1
 Title ""
-Date "12 oct 2015"
+Date "15 oct 2015"
 Rev ""
 Comp ""
@@
 Comment4 ""
 $EndDescr
+Connection ~ 7000 2550
+Wire Wire Line
+	7000 2300 7000 3050
+Wire Wire Line
+	7000 3050 7200 3050
 Wire Wire Line
 	1950 2900 1950 3000
@@
 	5600 3350 5600 3500
 Wire Wire Line
-	7200 3050 7200 3200
-Wire Wire Line
 	7850 4000 7850 4150
 Wire Wire Line
@@
 Wire Wire Line
 	5650 4200 5650 4050
-Wire Wire Line
-	6600 2500 6600 2600
 Wire Wire Line
 	6700 3100 6700 3300
@@
 Wire Wire Line
 	4900 2900 2550 2900
+Wire Wire Line
+	6600 2500 6600 2550
+Wire Wire Line
+	6600 2550 7000 2550
+$Comp
+L +3.3V #PWR?
+U 1 1 561F66DF
+P 7000 2300
+F 0 "#PWR?" H 7000 2260 30  0001 C CNN
+F 1 "+3.3V" H 7000 2410 30  0000 C CNN
+	1    7000 2300
+	1    0    0    -1
+$EndComp
 $Comp
 L GND #PWR01
@@
 $EndComp
 $Comp
-L GND #PWR03
-U 1 1 5612672C
-P 6600 2600
-F 0 "#PWR03" H 6600 2600 30  0001 C CNN
-F 1 "GND" H 6600 2530 30  0001 C CNN
-	1    6600 2600
-	1    0    0    -1
-$EndComp
-$Comp
 L R R8
 U 1 1 56126723
@@
 	1    0    0    -1
 $EndComp
-$Comp
-L GND #PWR07
-U 1 1 56126554
-P 7200 3200
-F 0 "#PWR07" H 7200 3200 30  0001 C CNN
-F 1 "GND" H 7200 3130 30  0001 C CNN
-	1    7200 3200
-	1    0    0    -1
-$EndComp
